File: pcb/v1.sch (EAGLE design)
At the start: 61 parts, among them T1 MMBT3904, T2 MMBT3904, T3 MMBT3904, T4 MMBT3904

Commit message: Changed PCB
Fixes #11
Fixes #10
Fixes #9
Fixes #8
Parts:
- removed 5V_TEST: PTR1B1,27, testpad:PTR1B1,27
- added C1, C2: 10uF, rcl:CPOL-USA/3216-18R
- added R17, R23: 10k, rcl:R-US_M1206
- added S1, S2: DTSM-6, switch-tact:DTSM-6
- added SW1: (no value), pinhead:PINHD-1X2
- added V_REG2: (no value), pinhead:PINHD-1X5
- C12, C13, C14, C15: value 10uF -> 22uF
- LED1, LED2, LED3, LED4: device led:LED5MM -> pinhead:PINHD-1X2
Connections:
- removed net N$11: LED3.C, R6.2
- new net LED3: LED3.2, R6.2
- new net N$22: C2.+, S2.4
- new net N$3: BATT1.1, SW1.1
- new net N$4: C1.+, S1.4
- new net SW1: C1.-, ESP32.IO23, R17.2, S1.1, S1.2
- new net SW2: C2.-, ESP32.IO27, R23.2, S2.1, S2.2
- net 3.3V: now also ESP32.IO0, S1.3, S2.3
- net 5V: now also LED1.1, LED2.1, LED3.1, LED4.1, V_REG2.5; no longer 5V_TEST.TP, LED1.A, LED2.A, LED3.A, LED4.A
- net BATT_POWER: now also SW1.2, V_REG2.1, V_REG2.2; no longer BATT1.1
- net EM1: now also ESP32.IO9; no longer ESP32.IO15
- net EM3: now also ESP32.IO14; no longer ESP32.IO0
- net EM4: now also ESP32.IO13; no longer ESP32.IO12
- net GND: now also R17.1, R23.1, V_REG2.3, V_REG2.4
- net N$14: now also LED4.2; no longer LED4.C
- net N$6: now also LED2.2; no longer LED1.C
- net N$8: now also LED1.2; no longer LED2.C
Other:
- moved on the sheet: BATT1, DRV1, DRV2, V_REG

Commit message: Cosmetic Changes
Connections:
- net BATT_POWER: now also C5.+, C7.+; no longer C5.-, C7.-
- net GND: now also C5.-, C7.-; no longer C5.+, C7.+
Other:
- moved on the sheet: C5, C7
Changed lines of the file:
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@@
 <part name="C5" library="rcl" library_urn="urn:adsk.eagle:library:334" deviceset="CPOL-US" device="150CLZ-0810" package3d_urn="urn:adsk.eagle:package:23394/2" value="47uF"/>
 <part name="X_13" library="ngspice-simulation" library_urn="urn:adsk.eagle:library:527439" deviceset="GND" device=""/>
-<part name="X_14" library="ngspice-simulation" library_urn="urn:adsk.eagle:library:527439" deviceset="GND" device=""/>
 <part name="R15" library="rcl" library_urn="urn:adsk.eagle:library:334" deviceset="R-US_" device="M1206" package3d_urn="urn:adsk.eagle:package:23566/2" value="30k"/>
 <part name="X_15" library="ngspice-simulation" library_urn="urn:adsk.eagle:library:527439" deviceset="GND" device=""/>
@@
 <part name="C7" library="rcl" library_urn="urn:adsk.eagle:library:334" deviceset="CPOL-US" device="150CLZ-0810" package3d_urn="urn:adsk.eagle:package:23394/2" value="47uF"/>
 <part name="X_17" library="ngspice-simulation" library_urn="urn:adsk.eagle:library:527439" deviceset="GND" device=""/>
-<part name="X_18" library="ngspice-simulation" library_urn="urn:adsk.eagle:library:527439" deviceset="GND" device=""/>
 <part name="R16" library="rcl" library_urn="urn:adsk.eagle:library:334" deviceset="R-US_" device="M1206" package3d_urn="urn:adsk.eagle:package:23566/2" value="30k"/>
 <part name="X_19" library="ngspice-simulation" library_urn="urn:adsk.eagle:library:527439" deviceset="GND" device=""/>
@@
 <attribute name="VALUE" x="37.211" y="178.816" size="1.778" layer="96" rot="R90"/>
 </instance>
-<instance part="C5" gate="G$1" x="27.94" y="185.42" smashed="yes">
-<attribute name="NAME" x="28.956" y="186.055" size="1.778" layer="95"/>
-<attribute name="VALUE" x="18.796" y="181.229" size="1.778" layer="96"/>
+<instance part="C5" gate="G$1" x="27.94" y="185.42" smashed="yes" rot="R180">
+<attribute name="NAME" x="26.924" y="184.785" size="1.778" layer="95" rot="R180"/>
+<attribute name="VALUE" x="37.084" y="189.611" size="1.778" layer="96" rot="R180"/>
 </instance>
 <instance part="X_13" gate="G$1" x="45.72" y="177.8" smashed="yes" rot="R90"/>
-<instance part="X_14" gate="G$1" x="27.94" y="193.04" smashed="yes" rot="R180"/>
 <instance part="R15" gate="G$1" x="-30.48" y="149.86" smashed="yes" rot="R90">
 <attribute name="NAME" x="-31.9786" y="148.59" size="1.778" layer="95" rot="R270"/>
@@
 <attribute name="VALUE" x="136.271" y="186.436" size="1.778" layer="96" rot="R90"/>
 </instance>
-<instance part="C7" gate="G$1" x="127" y="193.04" smashed="yes">
-<attribute name="NAME" x="128.016" y="193.675" size="1.778" layer="95"/>
-<attribute name="VALUE" x="117.856" y="188.849" size="1.778" layer="96"/>
+<instance part="C7" gate="G$1" x="127" y="193.04" smashed="yes" rot="R180">
+<attribute name="NAME" x="125.984" y="192.405" size="1.778" layer="95" rot="R180"/>
+<attribute name="VALUE" x="136.144" y="197.231" size="1.778" layer="96" rot="R180"/>
 </instance>
 <instance part="X_17" gate="G$1" x="144.78" y="185.42" smashed="yes" rot="R90"/>
-<instance part="X_18" gate="G$1" x="127" y="200.66" smashed="yes" rot="R180"/>
 <instance part="R16" gate="G$1" x="68.58" y="157.48" smashed="yes" rot="R90">
 <attribute name="NAME" x="67.0814" y="156.21" size="1.778" layer="95" rot="R270"/>
@@
 <pinref part="C4" gate="G$1" pin="+"/>
 <wire x1="27.94" y1="177.8" x2="30.48" y2="177.8" width="0.1524" layer="91"/>
-<pinref part="C5" gate="G$1" pin="-"/>
-<wire x1="27.94" y1="177.8" x2="27.94" y2="180.34" width="0.1524" layer="91"/>
 <label x="10.16" y="177.8" size="1.778" layer="95"/>
+<pinref part="C5" gate="G$1" pin="+"/>
+<wire x1="27.94" y1="177.8" x2="27.94" y2="182.88" width="0.1524" layer="91"/>
 </segment>
 <segment>
@@
 <pinref part="C6" gate="G$1" pin="+"/>
 <wire x1="127" y1="185.42" x2="129.54" y2="185.42" width="0.1524" layer="91"/>
-<pinref part="C7" gate="G$1" pin="-"/>
-<wire x1="127" y1="185.42" x2="127" y2="187.96" width="0.1524" layer="91"/>
 <label x="109.22" y="185.42" size="1.778" layer="95"/>
+<pinref part="C7" gate="G$1" pin="+"/>
+<wire x1="127" y1="185.42" x2="127" y2="190.5" width="0.1524" layer="91"/>
 </segment>
 <segment>
@@
 </segment>
 <segment>
-<pinref part="C5" gate="G$1" pin="+"/>
-<pinref part="X_14" gate="G$1" pin="0"/>
-<wire x1="27.94" y1="187.96" x2="27.94" y2="193.04" width="0.1524" layer="91"/>
-</segment>
-<segment>
 <pinref part="R15" gate="G$1" pin="1"/>
 <pinref part="X_15" gate="G$1" pin="0"/>
@@
 </segment>
 <segment>
-<pinref part="C7" gate="G$1" pin="+"/>
-<pinref part="X_18" gate="G$1" pin="0"/>
-<wire x1="127" y1="195.58" x2="127" y2="200.66" width="0.1524" layer="91"/>
-</segment>
-<segment>
 <pinref part="R16" gate="G$1" pin="1"/>
 <pinref part="X_19" gate="G$1" pin="0"/>
@@
 <label x="-5.08" y="220.98" size="1.778" layer="95"/>
 </segment>
-</net>
+<segment>
+<pinref part="C7" gate="G$1" pin="-"/>
+<wire x1="127" y1="198.12" x2="127" y2="200.66" width="0.1524" layer="91"/>
+<label x="127" y="200.66" size="1.778" layer="95"/>
+</segment>
+<segment>
+<pinref part="C5" gate="G$1" pin="-"/>
+<wire x1="27.94" y1="190.5" x2="27.94" y2="195.58" width="0.1524" layer="91"/>
+<label x="27.94" y="195.58" size="1.778" layer="95"/>
+</segment>
+</net>
