File: pcb/v1.brd (EAGLE design)
At the start: 92 x 80 mm, 68 parts, among them T1 MMBT3904, T2 MMBT3904, T3 MMBT3904, T4 MMBT3904

Commit message: blueberry: 📐
Routing:
- net BATT_POWER: track 146.0 -> 141.5 mm
Changed lines of the file:
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@@
 <wire x1="22.827825" y1="16.05118125" x2="24.24628125" y2="17.4696375" width="0.6096" layer="1"/>
 <wire x1="24.24628125" y1="17.4696375" x2="24.24628125" y2="17.770359375" width="0.6096" layer="1"/>
-<wire x1="11.488284375" y1="2.62924375" x2="11.6694375" y2="2.810396875" width="0.6096" layer="1"/>
-<wire x1="13.72081875" y1="11.176" x2="14.986" y2="11.176" width="0.6096" layer="1"/>
+<wire x1="14.986" y1="11.176" x2="13.72081875" y2="11.176" width="0.6096" layer="1"/>
 <via x="14.986" y="11.176" extent="1-16" drill="0.35"/>
 <wire x1="14.986" y1="11.176" x2="19.812" y2="11.176" width="0.6096" layer="16"/>
@@
 <wire x1="22.098" y1="13.462" x2="22.827825" y2="14.191825" width="0.6096" layer="1"/>
 <wire x1="22.827825" y1="14.191825" x2="22.827825" y2="16.05118125" width="0.6096" layer="1"/>
-<wire x1="5.323840625" y1="15.470215625" x2="5.323840625" y2="16.855440625" width="0.6096" layer="1"/>
 <wire x1="5.588" y1="33.213775" x2="9.458225" y2="33.213775" width="0.6096" layer="16"/>
 <wire x1="6.635" y1="39.125" x2="5.588" y2="38.078" width="0.6096" layer="1"/>
@@
 <wire x1="7.112" y1="18.6436" x2="7.112" y2="24.638" width="0.6096" layer="16"/>
 <wire x1="5.588" y1="26.162" x2="5.588" y2="33.02" width="0.6096" layer="16"/>
-<wire x1="14.218915625" y1="76.454" x2="14.32051875" y2="76.352396875" width="0.6096" layer="1"/>
-<wire x1="10.8013375" y1="76.454" x2="14.218915625" y2="76.454" width="0.6096" layer="1"/>
 <wire x1="14.32051875" y1="76.352396875" x2="16.86051875" y2="76.352396875" width="0.6096" layer="1"/>
 <wire x1="19.131" y1="69.197" x2="15.24" y2="69.197" width="0.6096" layer="1"/>
 <wire x1="16.86051875" y1="75.336396875" x2="16.86051875" y2="76.352396875" width="0.6096" layer="1"/>
 <wire x1="16.86051875" y1="75.336396875" x2="15.24" y2="73.715878125" width="0.6096" layer="1"/>
-<wire x1="15.24" y1="69.197" x2="15.24" y2="70.358" width="0.6096" layer="1"/>
-<wire x1="15.24" y1="70.358" x2="15.24" y2="73.715878125" width="0.6096" layer="1"/>
+<wire x1="15.24" y1="69.197" x2="15.24" y2="70.866" width="0.6096" layer="1"/>
+<wire x1="15.24" y1="70.866" x2="15.24" y2="73.715878125" width="0.6096" layer="1"/>
 <wire x1="16.61171875" y1="52.01905" x2="16.61171875" y2="49.8210625" width="0.3048" layer="1"/>
 <wire x1="16.61171875" y1="49.8210625" x2="17.0247875" y2="49.40799375" width="0.3048" layer="1"/>
@@
 <contactref element="C5" pad="+"/>
 <contactref element="C7" pad="+"/>
-<wire x1="15.24" y1="70.358" x2="11.77771875" y2="70.93038125" width="0.6096" layer="1"/>
-<wire x1="5.323840625" y1="16.855440625" x2="5.215528125" y2="11.432365625" width="0.6096" layer="1"/>
-<wire x1="5.215528125" y1="11.432365625" x2="5.1694375" y2="9.12461875" width="0.6096" layer="1"/>
-<wire x1="5.215528125" y1="11.432365625" x2="13.72081875" y2="11.176" width="0.6096" layer="1"/>
 <wire x1="11.488284375" y1="2.62924375" x2="5.1694375" y2="9.12461875" width="0.6096" layer="1"/>
+<wire x1="5.323840625" y1="16.855440625" x2="5.323840625" y2="9.279021875" width="0.508" layer="1"/>
+<wire x1="5.323840625" y1="9.279021875" x2="5.1694375" y2="9.12461875" width="0.508" layer="1"/>
+<wire x1="13.72081875" y1="11.176" x2="7.22081875" y2="11.176" width="0.508" layer="1"/>
+<wire x1="7.22081875" y1="11.176" x2="5.323840625" y2="9.279021875" width="0.508" layer="1"/>
+<wire x1="11.77771875" y1="70.93038125" x2="15.17561875" y2="70.93038125" width="0.508" layer="1"/>
+<wire x1="15.17561875" y1="70.93038125" x2="15.24" y2="70.866" width="0.508" layer="1"/>
 </signal>
 <signal name="N$1">
@@
 <contactref element="C7" pad="-"/>
 <contactref element="C5" pad="-"/>
-<wire x1="18.684" y1="71.708" x2="5.27771875" y2="70.93038125" width="0" layer="19" extent="1-1"/>
-<wire x1="11.6694375" y1="9.12461875" x2="13.946678125" y2="15.78864375" width="0" layer="19" extent="1-1"/>
 </signal>
 <signal name="N$5">

Commit message: Made connnecting grounds
Connections:
- net GND: no longer DRV1.P$1, DRV2.P$1, V_REG.P$1, V_REG.P$2
Changed lines of the file:
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@@
 <?xml version="1.0" encoding="utf-8"?>
 <!DOCTYPE eagle SYSTEM "eagle.dtd">
-<eagle version="9.4.0">
+<eagle version="9.3.0">
 <drawing>
 <settings>
@@
 <setting verticaltext="up"/>
 </settings>
-<grid distance="5" unitdist="mil" unit="mil" style="lines" multiple="1" display="yes" altdistance="5" altunitdist="mil" altunit="mil"/>
+<grid distance="5" unitdist="mil" unit="mil" style="lines" multiple="1" display="no" altdistance="1" altunitdist="mil" altunit="mil"/>
 <layers>
 <layer number="1" name="Top" color="4" fill="1" visible="yes" active="yes"/>
@@
 <layer number="24" name="bOrigins" color="15" fill="1" visible="yes" active="yes"/>
 <layer number="25" name="tNames" color="7" fill="1" visible="yes" active="yes"/>
-<layer number="26" name="bNames" color="7" fill="1" visible="no" active="yes"/>
-<layer number="27" name="tValues" color="7" fill="1" visible="no" active="yes"/>
-<layer number="28" name="bValues" color="7" fill="1" visible="no" active="yes"/>
-<layer number="29" name="tStop" color="7" fill="3" visible="yes" active="yes"/>
+<layer number="26" name="bNames" color="7" fill="1" visible="yes" active="yes"/>
+<layer number="27" name="tValues" color="7" fill="1" visible="yes" active="yes"/>
+<layer number="28" name="bValues" color="7" fill="1" visible="yes" active="yes"/>
+<layer number="29" name="tStop" color="7" fill="3" visible="no" active="yes"/>
 <layer number="30" name="bStop" color="7" fill="6" visible="no" active="yes"/>
 <layer number="31" name="tCream" color="7" fill="4" visible="no" active="yes"/>
@@
 <rectangle x1="80.899" y1="41.021" x2="82.677" y2="41.148" layer="1" rot="R90"/>
 <rectangle x1="81.026" y1="41.021" x2="82.296" y2="41.148" layer="1" rot="R90"/>
+<polygon width="0.1524" layer="30">
+<vertex x="20.574" y="68.707"/>
+<vertex x="22.606" y="68.707"/>
+<vertex x="22.606" y="65.913"/>
+<vertex x="20.574" y="65.913"/>
+</polygon>
+<polygon width="0.1524" layer="30">
+<vertex x="20.828" y="21.082"/>
+<vertex x="20.828" y="18.288"/>
+<vertex x="22.733" y="18.288"/>
+<vertex x="22.733" y="21.082"/>
+</polygon>
 </plain>
 <attributes>
@@
 </class>
 </classes>
-<designrules name="jlcpcb">
+<designrules name="jlcpcb *">
 <description language="de">&lt;b&gt;EAGLE Design Rules&lt;/b&gt;
 &lt;p&gt;
@@
 <param name="mtCopper" value="0.035mm 0.035mm 0.035mm 0.035mm 0.035mm 0.035mm 0.035mm 0.035mm 0.035mm 0.035mm 0.035mm 0.035mm 0.035mm 0.035mm 0.035mm 0.035mm"/>
 <param name="mtIsolate" value="1.5mm 0.15mm 0.2mm 0.15mm 0.2mm 0.15mm 0.2mm 0.15mm 0.2mm 0.15mm 0.2mm 0.15mm 0.2mm 0.15mm 0.2mm"/>
-<param name="mdWireWire" value="3.5mil"/>
+<param name="mdWireWire" value="5mil"/>
 <param name="mdWirePad" value="3.5mil"/>
 <param name="mdWireVia" value="5mil"/>
@@
 <param name="mdViaVia" value="6mil"/>
 <param name="mdSmdPad" value="6mil"/>
-<param name="mdSmdVia" value="6mil"/>
+<param name="mdSmdVia" value="0mil"/>
 <param name="mdSmdSmd" value="6mil"/>
 <param name="mdViaViaSameLayer" value="6mil"/>
 <param name="mnLayersViaInSmd" value="2"/>
-<param name="mdCopperDimension" value="0.2mm"/>
+<param name="mdCopperDimension" value="1mm"/>
 <param name="mdDrill" value="0.2mm"/>
 <param name="mdSmdStop" value="0mil"/>
@@
 <param name="msMicroVia" value="0.45mm"/>
 <param name="msBlindViaRatio" value="0.5"/>
-<param name="rvPadTop" value="0.25"/>
+<param name="rvPadTop" value="0.3"/>
 <param name="rvPadInner" value="0.25"/>
-<param name="rvPadBottom" value="0.25"/>
+<param name="rvPadBottom" value="0.3"/>
 <param name="rvViaOuter" value="0.25"/>
 <param name="rvViaInner" value="0.25"/>
@@
 <param name="checkNames" value="1"/>
 <param name="checkWireStubs" value="1"/>
-<param name="checkPolygonWidth" value="0"/>
+<param name="checkPolygonWidth" value="1"/>
 <param name="useDiameter" value="13"/>
 <param name="maxErrors" value="50"/>
@@
 <contactref element="V_REG2" pad="3"/>
 <contactref element="V_REG2" pad="4"/>
-<contactref element="DRV1" pad="P$1"/>
-<contactref element="DRV2" pad="P$1"/>
-<contactref element="V_REG" pad="P$1" route="any" routetag="G$1.PAD"/>
-<contactref element="V_REG" pad="P$2" route="any" routetag="G$1.PAD"/>
-<polygon width="0" layer="16">
-<vertex x="2.286" y="1.778"/>
-<vertex x="27.94" y="1.778"/>
-<vertex x="28.702" y="2.54"/>
-<vertex x="29.972" y="3.81"/>
-<vertex x="35.814" y="3.81"/>
-<vertex x="51.562" y="3.81"/>
-<vertex x="53.848" y="1.524"/>
-<vertex x="53.848" y="1.016"/>
-<vertex x="58.674" y="1.016"/>
-<vertex x="59.436" y="1.778"/>
-<vertex x="61.976" y="1.778"/>
-<vertex x="65.278" y="5.08"/>
-<vertex x="69.85" y="5.08"/>
-<vertex x="73.406" y="8.636"/>
-<vertex x="75.184" y="8.636"/>
-<vertex x="75.946" y="9.398"/>
-<vertex x="85.344" y="18.796"/>
-<vertex x="85.344" y="20.32"/>
-<vertex x="87.376" y="22.352"/>
-<vertex x="87.376" y="28.194"/>
-<vertex x="90.424" y="31.242"/>
-<vertex x="90.424" y="32.512"/>
-<vertex x="90.424" y="49.022"/>
-<vertex x="87.63" y="51.816"/>
-<vertex x="87.63" y="56.642"/>
-<vertex x="86.614" y="57.658"/>
-<vertex x="86.614" y="58.928"/>
-<vertex x="85.852" y="59.69"/>
-<vertex x="85.852" y="60.96"/>
-<vertex x="81.026" y="65.786"/>
-<vertex x="81.026" y="66.294"/>
-<vertex x="75.184" y="72.136"/>
-<vertex x="71.628" y="72.136"/>
-<vertex x="67.564" y="76.2"/>
-<vertex x="66.04" y="76.2"/>
-<vertex x="64.516" y="77.724"/>
-<vertex x="57.912" y="77.724"/>
-<vertex x="56.134" y="79.502"/>
-<vertex x="52.832" y="79.502"/>
-<vertex x="52.832" y="77.47"/>
-<vertex x="51.054" y="75.692"/>
-<vertex x="30.734" y="75.692"/>
-<vertex x="30.226" y="76.2"/>
-<vertex x="27.686" y="78.74"/>
-<vertex x="27.686" y="79.502"/>
-<vertex x="4.826" y="79.502"/>
-<vertex x="4.572" y="79.756"/>
-<vertex x="4.318" y="79.502"/>
-<vertex x="0.762" y="79.502"/>
-<vertex x="0.762" y="2.794"/>
-<vertex x="1.27" y="2.286"/>
-<vertex x="1.778" y="1.778"/>
-</polygon>
-<polygon width="0" layer="1">
-<vertex x="0.508" y="27.686"/>
-<vertex x="0.508" y="2.794"/>
-<vertex x="1.778" y="1.524"/>
-<vertex x="27.94" y="1.524"/>
-<vertex x="28.702" y="2.286"/>
-<vertex x="29.972" y="3.556"/>
-<vertex x="29.972" y="3.81"/>
-<vertex x="51.816" y="3.81"/>
-<vertex x="54.356" y="1.27"/>
-<vertex x="54.356" y="1.016"/>
-<vertex x="59.944" y="1.016"/>
-<vertex x="64.262" y="5.334"/>
-<vertex x="68.072" y="5.334"/>
-<vertex x="77.978" y="15.24"/>
-<vertex x="81.026" y="15.24"/>
-<vertex x="86.614" y="20.828"/>
-<vertex x="86.614" y="24.638"/>
-<vertex x="89.662" y="27.686"/>
-<vertex x="89.662" y="34.798"/>
-<vertex x="89.662" y="49.022"/>
-<vertex x="87.63" y="51.054"/>
-<vertex x="87.63" y="56.896"/>
-<vertex x="83.312" y="61.214"/>
-<vertex x="83.312" y="63.5"/>
-<vertex x="80.518" y="66.294"/>
-<vertex x="75.184" y="71.628"/>
-<vertex x="72.898" y="71.628"/>
-<vertex x="68.326" y="76.2"/>
-<vertex x="63.754" y="76.2"/>
-<vertex x="61.722" y="78.232"/>
-<vertex x="55.626" y="78.232"/>
-<vertex x="53.34" y="78.232"/>
-<vertex x="51.816" y="76.708"/>
-<vertex x="51.308" y="76.2"/>
-<vertex x="51.308" y="75.692"/>
-<vertex x="30.988" y="75.692"/>
-<vertex x="27.178" y="79.502"/>
-<vertex x="26.416" y="79.502"/>
-<vertex x="1.016" y="79.502"/>
-<vertex x="0.508" y="78.994"/>
-</polygon>
 <contactref element="C7" pad="-"/>
 <contactref element="C5" pad="-"/>
+<polygon width="0.1524" layer="1" thermals="no">
+<vertex x="0" y="78.9746"/>
+<vertex x="0" y="0.9746" curve="90"/>
+<vertex x="1" y="-0.0254"/>
+<vertex x="52" y="-0.0254" curve="180"/>
+<vertex x="52" y="79.9746"/>
+<vertex x="1" y="79.9746" curve="90"/>
+</polygon>
+<polygon width="0.1524" layer="16" thermals="no">
+<vertex x="0" y="78.9746"/>
+<vertex x="0" y="0.9746" curve="90"/>
+<vertex x="1" y="-0.0254"/>
+<vertex x="52" y="-0.0254" curve="180"/>
+<vertex x="52" y="79.9746"/>
+<vertex x="1" y="79.9746" curve="90"/>
+</polygon>
+<via x="21.082" y="68.072" extent="1-16" drill="0.35"/>
+<via x="22.098" y="68.072" extent="1-16" drill="0.35"/>
+<via x="21.082" y="67.31" extent="1-16" drill="0.35"/>
+<via x="22.098" y="67.31" extent="1-16" drill="0.35"/>
+<via x="22.098" y="66.548" extent="1-16" drill="0.35"/>
+<via x="21.082" y="66.548" extent="1-16" drill="0.35"/>
+<via x="21.336" y="20.574" extent="1-16" drill="0.35"/>
+<via x="22.352" y="20.574" extent="1-16" drill="0.35"/>
+<via x="21.336" y="19.812" extent="1-16" drill="0.35"/>
+<via x="22.352" y="19.812" extent="1-16" drill="0.35"/>
+<via x="21.336" y="19.05" extent="1-16" drill="0.35"/>
+<via x="22.352" y="19.05" extent="1-16" drill="0.35"/>
+<via x="5.08" y="42.672" extent="1-16" drill="0.35"/>
+<via x="6.096" y="42.672" extent="1-16" drill="0.35"/>
+<via x="7.112" y="42.672" extent="1-16" drill="0.35"/>
+<via x="5.08" y="41.402" extent="1-16" drill="0.35"/>
+<via x="6.096" y="41.402" extent="1-16" drill="0.35"/>
+<via x="7.112" y="41.402" extent="1-16" drill="0.35"/>
+<via x="42.799" y="73.152" extent="1-16" drill="0.35"/>
 </signal>
 <signal name="N$5">
@@
 <via x="83.82" y="44.323" extent="1-16" drill="0.35"/>
 </signal>
+<signal name="GND1" airwireshidden="yes">
+<via x="44.069" y="13.589" extent="1-16" drill="0.35"/>
+</signal>
+<signal name="GND2" airwireshidden="yes">
+<via x="44.45" y="8.509" extent="1-16" drill="0.35"/>
+</signal>
+<signal name="GND3" airwireshidden="yes">
+<via x="52.959" y="38.989" extent="1-16" drill="0.35"/>
+</signal>
+<signal name="GND4" airwireshidden="yes">
+<via x="23.876" y="38.481" extent="1-16" drill="0.35"/>
+</signal>
+<signal name="GND5" airwireshidden="yes">
+<via x="10.287" y="23.876" extent="1-16" drill="0.35"/>
+</signal>
 </signals>
